File: Kicad-Main/xbee-node-attiny841.sch (KiCad schematic (older format))
At the start: 36 parts, among them P10 CONN_1, P11 CONN_1, P12 CONN_1, P13 CONN_1, P14 CONN_1, P15 CONN_1, P16 CONN_1, P17 CONN_1, P18 CONN_1, P2 XBee Adaptor, P3 Test, P4 Battery, P5 XBee-ext-1, P6 XBee-ext-2, P7 CONN_1, P8 CONN_1, P9 CONN_1, Q1 S1133, Q2 S9014, Q3 2N7000, U1 ATTINY84-S, U2 MAX952ESA, U3 TPS77033

Commit message: Modification of boards after checking. Addition of other LED types to LED mount board.
Parts:
- U1: footprint SMD_Packages:SOIC-14_N -> Photodiode:ATTINY841-SSU
Connections:
- no-connect marks 7 -> 6
Changed lines of the file:
@@
 LIBS:contrib
 LIBS:valves
-LIBS:RF_OEM_Parts
-LIBS:KB1LQC
 LIBS:xbee-node-attiny841-cache
 EELAYER 24 0
@@
 	1    0    0    -1
 $EndComp
-Text Label 9650 2000 0    60   ~ 0
+Text Label 9650 2500 0    60   ~ 0
 VBatt
 Text Label 7650 4550 0    60   ~ 0
@@
 F 0 "U1" H 2550 4150 40  0000 C CNN
 F 1 "ATTINY84-S" H 4100 2650 40  0000 C CNN
-F 2 "SMD_Packages:SOIC-14_N" H 3400 3200 35  0000 C CIN
+F 2 "Photodiode:ATTINY841-SSU" H 3400 3200 35  0000 C CIN
 F 3 "" H 3400 3400 60  0000 C CNN
 	1    3400 3400
@@
 Text Label 8950 5300 2    60   ~ 0
 Bootloader
-NoConn ~ 8950 5100
 NoConn ~ 8950 5200
 $Comp
@@
 	1    0    0    -1
 $EndComp
+$Comp
+L GND #PWR?
+U 1 1 53FEF658
+P 8950 5100
+F 0 "#PWR?" H 8950 5100 30  0001 C CNN
+F 1 "GND" H 8950 5030 30  0001 C CNN
+F 2 "" H 8950 5100 60  0000 C CNN
+F 3 "" H 8950 5100 60  0000 C CNN
+	1    8950 5100
+	0    1    -1   0
+$EndComp
 $EndSCHEMATC

Commit message: Change schematic symbols for connectors as Kicad, inexplicably, removed them.
Parts:
- P10, P11, P12, P13, P14, P15, P16, P17, P18, P7, P8, P9: symbol CONN_1 -> CONN_01X01
- P2: symbol CONN_6X2 -> CONN_02X06
- P3: symbol CONN_5X2 -> CONN_02X05
- P4: symbol CONN_2 -> CONN_01X02
- P5, P6: symbol CONN_3 -> CONN_01X03
Changed lines of the file:
@@
 LIBS:contrib
 LIBS:valves
-LIBS:xbee-node-attiny841-cache
+LIBS:DataStorage
+LIBS:RF_OEM_Parts
+LIBS:KB1LQC
+LIBS:MiscellaneousDevices
+LIBS:TransistorParts
+LIBS:Sensors
 EELAYER 24 0
 EELAYER END
@@
 $EndDescr
 $Comp
-L CONN_2 P4
+L CONN_01X02 P4
 U 1 1 53D32A7E
-P 10400 1500
-F 0 "P4" V 10350 1500 40  0000 C CNN
-F 1 "Battery" V 10450 1500 40  0000 C CNN
-F 2 "Connect:SIL-2" H 10400 1500 60  0001 C CNN
-F 3 "" H 10400 1500 60  0000 C CNN
-	1    10400 1500
+P 10250 1450
+F 0 "P4" V 10200 1450 40  0000 C CNN
+F 1 "Battery" V 10300 1450 40  0000 C CNN
+F 2 "Connect:SIL-2" H 10250 1450 60  0001 C CNN
+F 3 "" H 10250 1450 60  0000 C CNN
+	1    10250 1450
 	1    0    0    -1
 $EndComp
@@
 L VDD #PWR011
 U 1 1 53D35928
-P 7650 4450
-F 0 "#PWR011" H 7650 4550 30  0001 C CNN
-F 1 "VDD" H 7650 4560 30  0000 C CNN
-F 2 "" H 7650 4450 60  0000 C CNN
-F 3 "" H 7650 4450 60  0000 C CNN
-	1    7650 4450
+P 7500 4450
+F 0 "#PWR011" H 7500 4550 30  0001 C CNN
+F 1 "VDD" H 7500 4560 30  0000 C CNN
+F 2 "" H 7500 4450 60  0000 C CNN
+F 3 "" H 7500 4450 60  0000 C CNN
+	1    7500 4450
 	0    1    1    0
 $EndComp
@@
 	1    0    0    -1
 $EndComp
-Text Label 6850 4850 2    60   ~ 0
+Text Label 7000 4850 2    60   ~ 0
 On/Sleep
 Text Label 4450 2800 0    60   ~ 0
@@
 Text Label 4450 3700 0    60   ~ 0
 Bootloader
-Text Label 7650 4950 0    60   ~ 0
+Text Label 7500 4950 0    60   ~ 0
 Tx
-Text Label 6850 4750 2    60   ~ 0
+Text Label 7000 4750 2    60   ~ 0
 Rx
 Text Label 4450 3000 0    60   ~ 0
@@
 Tx
 $Comp
-L CONN_6X2 P2
+L CONN_02X06 P2
 U 1 1 53DDD3EB
 P 7250 4700
@@
 Text Label 9650 2500 0    60   ~ 0
 VBatt
-Text Label 7650 4550 0    60   ~ 0
+Text Label 7500 4550 0    60   ~ 0
 VBatt
 Text Label 1450 3500 0    60   ~ 0
 Reset
-Text Label 6850 4650 2    60   ~ 0
+Text Label 7000 4650 2    60   ~ 0
 Reset
 $Comp
@@
 $EndComp
 $Comp
-L CONN_5X2 P3
+L CONN_02X05 P3
 U 1 1 53E0177A
 P 7250 5700
@@
 L GND #PWR019
 U 1 1 53E0741A
-P 6850 5900
-F 0 "#PWR019" H 6850 5900 30  0001 C CNN
-F 1 "GND" H 6850 5830 30  0001 C CNN
-F 2 "" H 6850 5900 60  0000 C CNN
-F 3 "" H 6850 5900 60  0000 C CNN
-	1    6850 5900
+P 7000 5900
+F 0 "#PWR019" H 7000 5900 30  0001 C CNN
+F 1 "GND" H 7000 5830 30  0001 C CNN
+F 2 "" H 7000 5900 60  0000 C CNN
+F 3 "" H 7000 5900 60  0000 C CNN
+	1    7000 5900
 	0    1    -1   0
 $EndComp
-Text Label 7650 5500 0    60   ~ 0
+Text Label 7500 5500 0    60   ~ 0
 VBatt
 $Comp
@@
 L GND #PWR026
 U 1 1 53E22A19
-P 6850 4950
-F 0 "#PWR026" H 6850 4950 30  0001 C CNN
-F 1 "GND" H 6850 4880 30  0001 C CNN
-F 2 "" H 6850 4950 60  0000 C CNN
-F 3 "" H 6850 4950 60  0000 C CNN
-	1    6850 4950
+P 7000 4950
+F 0 "#PWR026" H 7000 4950 30  0001 C CNN
+F 1 "GND" H 7000 4880 30  0001 C CNN
+F 2 "" H 7000 4950 60  0000 C CNN
+F 3 "" H 7000 4950 60  0000 C CNN
+	1    7000 4950
 	0    1    -1   0
 $EndComp
@@
 L GND #PWR027
 U 1 1 53E26458
-P 10050 1600
-F 0 "#PWR027" H 10050 1600 30  0001 C CNN
-F 1 "GND" H 10050 1530 30  0001 C CNN
-F 2 "" H 10050 1600 60  0000 C CNN
-F 3 "" H 10050 1600 60  0000 C CNN
-	1    10050 1600
+P 10050 1500
+F 0 "#PWR027" H 10050 1500 30  0001 C CNN
+F 1 "GND" H 10050 1430 30  0001 C CNN
+F 2 "" H 10050 1500 60  0000 C CNN
+F 3 "" H 10050 1500 60  0000 C CNN
+	1    10050 1500
 	0    1    1    0
 $EndComp
@@
 Text Label 4450 3400 0    60   ~ 0
 MOSI
-Text Label 7650 5700 0    60   ~ 0
+Text Label 7500 5700 0    60   ~ 0
 SCK
-Text Label 6850 5700 2    60   ~ 0
+Text Label 7000 5700 2    60   ~ 0
 MISO
-Text Label 6850 5600 2    60   ~ 0
+Text Label 7000 5600 2    60   ~ 0
 MOSI
-NoConn ~ 6850 4450
-NoConn ~ 7650 4850
+NoConn ~ 7000 4450
+NoConn ~ 7500 4850
 $Comp
 L C C6
@@
 Connection ~ 5650 1550
 Connection ~ 5400 1550
-Text Label 7650 5600 0    60   ~ 0
+Text Label 7500 5600 0    60   ~ 0
 Reset
-Text Label 6850 5800 2    60   ~ 0
+Text Label 7000 5800 2    60   ~ 0
 Rx
-Text Label 7650 5800 0    60   ~ 0
+Text Label 7500 5800 0    60   ~ 0
 Tx
 Connection ~ 4450 5600
@@
 Text Label 4450 5600 0    60   ~ 0
 Count
-Text Label 6850 5500 2    60   ~ 0
+Text Label 7000 5500 2    60   ~ 0
 Count
-Text Label 7650 4650 0    60   ~ 0
+Text Label 7500 4650 0    60   ~ 0
 Xbee-Reset
-Text Label 7650 4750 0    60   ~ 0
+Text Label 7500 4750 0    60   ~ 0
 Sleep-Rq
-Text Label 6850 4550 2    60   ~ 0
+Text Label 7000 4550 2    60   ~ 0
 Bootloader
-Text Label 7650 5900 0    60   ~ 0
+Text Label 7500 5900 0    60   ~ 0
 On/Sleep
 $Comp
-L CONN_3 P5
+L CONN_01X03 P5
 U 1 1 53F2B594
-P 9300 4650
-F 0 "P5" H 9300 4850 50  0000 C CNN
-F 1 "XBee-ext-1" V 9450 4650 40  0000 C CNN
-F 2 "Photodiode:pin_header_2mm_1x3" H 9300 4650 60  0001 C CNN
-F 3 "" H 9300 4650 60  0000 C CNN
-	1    9300 4650
-	1    0    0    -1
-$EndComp
-$Comp
-L CONN_3 P6
+P 9150 4650
+F 0 "P5" H 9150 4850 50  0000 C CNN
+F 1 "XBee-ext-1" V 9300 4650 40  0000 C CNN
+F 2 "Photodiode:pin_header_2mm_1x3" H 9150 4650 60  0001 C CNN
+F 3 "" H 9150 4650 60  0000 C CNN
+	1    9150 4650
+	1    0    0    -1
+$EndComp
+$Comp
+L CONN_01X03 P6
 U 1 1 53F2B605
-P 9300 5200
-F 0 "P6" H 9300 5400 50  0000 C CNN
-F 1 "XBee-ext-2" V 9450 5200 40  0000 C CNN
-F 2 "Photodiode:pin_header_2mm_1x3" H 9300 5200 60  0001 C CNN
-F 3 "" H 9300 5200 60  0000 C CNN
-	1    9300 5200
+P 9150 5200
+F 0 "P6" H 9150 5400 50  0000 C CNN
+F 1 "XBee-ext-2" V 9300 5200 40  0000 C CNN
+F 2 "Photodiode:pin_header_2mm_1x3" H 9150 5200 60  0001 C CNN
+F 3 "" H 9150 5200 60  0000 C CNN
+	1    9150 5200
 	1    0    0    -1
 $EndComp
@@
 NoConn ~ 8950 5200
 $Comp
-L CONN_1 P7
+L CONN_01X01 P7
 U 1 1 53F2CFA4
 P 8700 1900
@@
 $EndComp
 $Comp
-L CONN_1 P8
+L CONN_01X01 P8
 U 1 1 53F2D10A
 P 8600 1900
@@
 $EndComp
 $Comp
-L CONN_1 P9
+L CONN_01X01 P9
 U 1 1 53F2D15D
 P 8500 1900
@@
 $EndComp
 $Comp
-L CONN_1 P10
+L CONN_01X01 P10
 U 1 1 53F32A4A
 P 7900 1950
@@
 $EndComp
 $Comp
-L CONN_1 P11
+L CONN_01X01 P11
 U 1 1 53F32AA5
 P 8050 1950
@@
 PowerControl
 $Comp
-L CONN_1 P12
+L CONN_01X01 P12
 U 1 1 53F2D7DC
 P 7550 2350
@@
 $EndComp
 $Comp
-L CONN_1 P13
+L CONN_01X01 P13
 U 1 1 53F2D842
 P 7700 2350
@@
 $EndComp
 $Comp
-L CONN_1 P14
+L CONN_01X01 P14
 U 1 1 53F2D878
 P 7850 2350
@@
 $EndComp
 $Comp
-L CONN_1 P15
+L CONN_01X01 P15
 U 1 1 53F2D8B3
 P 8000 2350
@@
 $EndComp
 $Comp
-L CONN_1 P16
+L CONN_01X01 P16
 U 1 1 53F2DBA5
 P 8200 2350
@@
 $EndComp
 $Comp
-L CONN_1 P17
+L CONN_01X01 P17
 U 1 1 53F2DBF0
 P 8350 2350
@@
 $EndComp
 $Comp
-L CONN_1 P18
+L CONN_01X01 P18
 U 1 1 53F2DF81
 P 8500 2350

Commit message: Correct some wiring and ground connection errors in the main board PCB. Reduce size of the LED mount to fit inside meter.
Parts:
- removed Q1: S1133, PhotoDiode:S1133TH, symbol OPTO_NPN
- added D2: S1133, Photodiode:S1133TH, symbol PHOTODIODE
- D1: value APD3224ZGC-F01 -> SFH4056
Connections:
- net labels added: Battery
- wire segments 13 -> 17
Other:
- moved on the sheet: U1

Commit message: Main board add pulldown to XBee-sleep line.
Parts:
- added R9: 1M, SMD_Packages:SM0603_Resistor, symbol R
Changed lines of the file:
@@
 $EndComp
 $Comp
-L GND #PWR030
+L GND #PWR029
 U 1 1 53E234F6
 P 5650 1950
-F 0 "#PWR030" H 5650 1950 30  0001 C CNN
+F 0 "#PWR029" H 5650 1950 30  0001 C CNN
 F 1 "GND" H 5650 1880 30  0001 C CNN
 F 2 "" H 5650 1950 60  0000 C CNN
@@
 $EndComp
 $Comp
-L GND #PWR031
+L GND #PWR030
 U 1 1 53E2398F
 P 5900 1950
-F 0 "#PWR031" H 5900 1950 30  0001 C CNN
+F 0 "#PWR030" H 5900 1950 30  0001 C CNN
 F 1 "GND" H 5900 1880 30  0001 C CNN
 F 2 "" H 5900 1950 60  0000 C CNN
@@
 $EndComp
 $Comp
-L GND #PWR032
+L GND #PWR031
 U 1 1 53F32D83
 P 7900 2150
-F 0 "#PWR032" H 7900 2150 30  0001 C CNN
+F 0 "#PWR031" H 7900 2150 30  0001 C CNN
 F 1 "GND" H 7900 2080 30  0001 C CNN
 F 2 "" H 7900 2150 60  0000 C CNN
@@
 $EndComp
 $Comp
-L GND #PWR033
+L GND #PWR032
 U 1 1 53F32DAC
 P 8050 2150
-F 0 "#PWR033" H 8050 2150 30  0001 C CNN
+F 0 "#PWR032" H 8050 2150 30  0001 C CNN
 F 1 "GND" H 8050 2080 30  0001 C CNN
 F 2 "" H 8050 2150 60  0000 C CNN
@@
 $EndComp
 $Comp
-L GND #PWR034
+L GND #PWR033
 U 1 1 53F2D923
 P 7550 2550
-F 0 "#PWR034" H 7550 2550 30  0001 C CNN
+F 0 "#PWR033" H 7550 2550 30  0001 C CNN
 F 1 "GND" H 7550 2480 30  0001 C CNN
 F 2 "" H 7550 2550 60  0000 C CNN
@@
 $EndComp
 $Comp
-L GND #PWR035
+L GND #PWR034
 U 1 1 53F2D950
 P 7700 2550
-F 0 "#PWR035" H 7700 2550 30  0001 C CNN
+F 0 "#PWR034" H 7700 2550 30  0001 C CNN
 F 1 "GND" H 7700 2480 30  0001 C CNN
 F 2 "" H 7700 2550 60  0000 C CNN
@@
 $EndComp
 $Comp
-L GND #PWR036
+L GND #PWR035
 U 1 1 53F2D99F
 P 7850 2550
-F 0 "#PWR036" H 7850 2550 30  0001 C CNN
+F 0 "#PWR035" H 7850 2550 30  0001 C CNN
 F 1 "GND" H 7850 2480 30  0001 C CNN
 F 2 "" H 7850 2550 60  0000 C CNN
@@
 $EndComp
 $Comp
-L GND #PWR037
+L GND #PWR036
 U 1 1 53F2D9CC
 P 8000 2550
-F 0 "#PWR037" H 8000 2550 30  0001 C CNN
+F 0 "#PWR036" H 8000 2550 30  0001 C CNN
 F 1 "GND" H 8000 2480 30  0001 C CNN
 F 2 "" H 8000 2550 60  0000 C CNN
@@
 $EndComp
 $Comp
-L GND #PWR038
+L GND #PWR037
 U 1 1 53F2DC2E
 P 8200 2550
-F 0 "#PWR038" H 8200 2550 30  0001 C CNN
+F 0 "#PWR037" H 8200 2550 30  0001 C CNN
 F 1 "GND" H 8200 2480 30  0001 C CNN
 F 2 "" H 8200 2550 60  0000 C CNN
@@
 $EndComp
 $Comp
-L GND #PWR039
+L GND #PWR038
 U 1 1 53F2DC5D
 P 8350 2550
-F 0 "#PWR039" H 8350 2550 30  0001 C CNN
+F 0 "#PWR038" H 8350 2550 30  0001 C CNN
 F 1 "GND" H 8350 2480 30  0001 C CNN
 F 2 "" H 8350 2550 60  0000 C CNN
@@
 $EndComp
 $Comp
-L GND #PWR040
+L GND #PWR039
 U 1 1 53F2DFE3
 P 8500 2550
-F 0 "#PWR040" H 8500 2550 30  0001 C CNN
+F 0 "#PWR039" H 8500 2550 30  0001 C CNN
 F 1 "GND" H 8500 2480 30  0001 C CNN
 F 2 "" H 8500 2550 60  0000 C CNN
@@
 $EndComp
 $Comp
-L GND #PWR041
+L GND #PWR040
 U 1 1 53FEF658
 P 8950 5100
-F 0 "#PWR041" H 8950 5100 30  0001 C CNN
+F 0 "#PWR040" H 8950 5100 30  0001 C CNN
 F 1 "GND" H 8950 5030 30  0001 C CNN
 F 2 "" H 8950 5100 60  0000 C CNN
@@
 Wire Wire Line
 	10050 1500 9950 1500
+$Comp
+L R R9
+U 1 1 54823620
+P 7000 3000
+F 0 "R9" V 7080 3000 40  0000 C CNN
+F 1 "1M" V 7007 3001 40  0000 C CNN
+F 2 "SMD_Packages:SM0603_Resistor" V 6930 3000 30  0001 C CNN
+F 3 "" H 7000 3000 30  0000 C CNN
+	1    7000 3000
+	-1   0    0    1
+$EndComp
+$Comp
+L GND #PWR041
+U 1 1 5482395B
+P 7000 3250
+F 0 "#PWR041" H 7000 3250 30  0001 C CNN
+F 1 "GND" H 7000 3180 30  0001 C CNN
+F 2 "" H 7000 3250 60  0000 C CNN
+F 3 "" H 7000 3250 60  0000 C CNN
+	1    7000 3250
+	1    0    0    -1
+$EndComp
+Text Label 7000 2750 0    60   ~ 0
+Sleep-Rq
 $EndSCHEMATC

Commit message: Update main board to filter analogue power runs and shield input signals.
Parts:
- added C8, C9: 0.1uF, SMD_Packages:SMD-0603_c, symbol C
- added L1: INDUCTOR_SMALL, Resistors_SMD:R_0603, symbol INDUCTOR_SMALL
Connections:
- net labels added: VDDA
- wire segments 17 -> 20

Commit message: Minor change to board schematic to put capacitor on correct power line.
Other:
- moved on the sheet: L1
Changed lines of the file:
@@
 L C C6
 U 1 1 53E234F0
-P 5650 1750
-F 0 "C6" H 5650 1850 40  0000 L CNN
-F 1 "0.1uF" H 5656 1665 40  0000 L CNN
-F 2 "SMD_Packages:SM0603_Capa" H 5688 1600 30  0001 C CNN
-F 3 "" H 5650 1750 60  0000 C CNN
-	1    5650 1750
+P 4150 1750
+F 0 "C6" H 4150 1850 40  0000 L CNN
+F 1 "0.1uF" H 4156 1665 40  0000 L CNN
+F 2 "SMD_Packages:SM0603_Capa" H 4188 1600 30  0001 C CNN
+F 3 "" H 4150 1750 60  0000 C CNN
+	1    4150 1750
 	1    0    0    -1
 $EndComp
@@
 L GND #PWR024
 U 1 1 53E234F6
-P 5650 1950
-F 0 "#PWR024" H 5650 1950 30  0001 C CNN
-F 1 "GND" H 5650 1880 30  0001 C CNN
-F 2 "" H 5650 1950 60  0000 C CNN
-F 3 "" H 5650 1950 60  0000 C CNN
-	1    5650 1950
+P 4150 1950
+F 0 "#PWR024" H 4150 1950 30  0001 C CNN
+F 1 "GND" H 4150 1880 30  0001 C CNN
+F 2 "" H 4150 1950 60  0000 C CNN
+F 3 "" H 4150 1950 60  0000 C CNN
+	1    4150 1950
 	1    0    0    -1
 $EndComp
@@
 L INDUCTOR_SMALL L1
 U 1 1 548D0C86
-P 4550 1550
-F 0 "L1" H 4550 1650 50  0000 C CNN
-F 1 "INDUCTOR_SMALL" H 4550 1500 50  0000 C CNN
-F 2 "Resistors_SMD:R_0603" H 4550 1550 60  0001 C CNN
-F 3 "" H 4550 1550 60  0000 C CNN
-	1    4550 1550
+P 4800 1550
+F 0 "L1" H 4800 1650 50  0000 C CNN
+F 1 "INDUCTOR_SMALL" H 4800 1500 50  0000 C CNN
+F 2 "Resistors_SMD:R_0603" H 4800 1550 60  0001 C CNN
+F 3 "" H 4800 1550 60  0000 C CNN
+	1    4800 1550
 	1    0    0    -1
 $EndComp
@@
 L C C9
 U 1 1 548D1179
-P 4150 1750
-F 0 "C9" H 4150 1850 40  0000 L CNN
-F 1 "0.1uF" H 4156 1665 40  0000 L CNN
-F 2 "SMD_Packages:SMD-0603_c" H 4188 1600 30  0001 C CNN
-F 3 "" H 4150 1750 60  0000 C CNN
-	1    4150 1750
+P 4450 1750
+F 0 "C9" H 4450 1850 40  0000 L CNN
+F 1 "0.1uF" H 4456 1665 40  0000 L CNN
+F 2 "SMD_Packages:SMD-0603_c" H 4488 1600 30  0001 C CNN
+F 3 "" H 4450 1750 60  0000 C CNN
+	1    4450 1750
 	1    0    0    -1
 $EndComp
@@
 L GND #PWR038
 U 1 1 548D117F
-P 4150 1950
-F 0 "#PWR038" H 4150 1950 30  0001 C CNN
-F 1 "GND" H 4150 1880 30  0001 C CNN
-F 2 "" H 4150 1950 60  0000 C CNN
-F 3 "" H 4150 1950 60  0000 C CNN
-	1    4150 1950
+P 4450 1950
+F 0 "#PWR038" H 4450 1950 30  0001 C CNN
+F 1 "GND" H 4450 1880 30  0001 C CNN
+F 2 "" H 4450 1950 60  0000 C CNN
+F 3 "" H 4450 1950 60  0000 C CNN
+	1    4450 1950
 	1    0    0    -1
 $EndComp
@@
 Connection ~ 6150 1550
 Connection ~ 5900 1550
-Connection ~ 5650 1550
+Connection ~ 4450 1550
 Connection ~ 5400 1550
 Connection ~ 5950 5250
@@
 	10050 1500 9950 1500
 Wire Wire Line
-	4800 1550 6300 1550
-Wire Wire Line
-	4000 1550 4300 1550
+	5050 1550 6300 1550
+Wire Wire Line
+	4000 1550 4550 1550
 Connection ~ 5100 1550
 Wire Wire Line
@@
 Text Label 4100 4450 1    60   ~ 0
 VDDA
+Connection ~ 6900 1400
+Connection ~ 6300 1550
 $EndSCHEMATC
