File: Kicad-Main/xbee-node-attiny841.sch (KiCad schematic (older format))
At the start: 40 parts, among them P10 CONN_1, P11 CONN_1, P12 CONN_1, P13 CONN_1, P14 CONN_1, P15 CONN_1, P16 CONN_1, P17 CONN_1, P18 CONN_1, P2 XBee Adaptor, P3 Test, P4 Battery, P5 XBee-ext-1, P6 XBee-ext-2, P7 CONN_1, P8 CONN_1, P9 CONN_1, Q2 S9014, Q3 2N7000, U1 ATTINY84-S, U2 MAX952ESA, U3 TPS77033

Commit message: Main board: add a regulator for the XBee power only, plus capacitor.
Parts:
- added C10: 3.3uF, SMD_Packages:SMD-1206_Pol, symbol CP
- added P19: CONN_1, Photodiode:THROUGHVIA, symbol CONN_01X01
- added U4: TPS77033, SMD_Packages:SOT-23-5, symbol TPS77033
Connections:
- net labels added: VDDX
- wire segments 20 -> 23
- no-connect marks 6 -> 7
Changed lines of the file:
@@
-$EndComp
-$Comp
-L VDD #PWR011
-U 1 1 53D35928
-P 7500 4450
-F 0 "#PWR011" H 7500 4550 30  0001 C CNN
-F 1 "VDD" H 7500 4560 30  0000 C CNN
-F 2 "" H 7500 4450 60  0000 C CNN
-F 3 "" H 7500 4450 60  0000 C CNN
-	1    7500 4450
-	0    1    1    0
 $EndComp
 $Comp
@@
 $EndComp
 $Comp
-L GND #PWR012
+L GND #PWR011
 U 1 1 53D35BB6
 P 5350 5650
-F 0 "#PWR012" H 5350 5650 30  0001 C CNN
+F 0 "#PWR011" H 5350 5650 30  0001 C CNN
 F 1 "GND" H 5350 5580 30  0001 C CNN
 F 2 "" H 5350 5650 60  0000 C CNN
@@
 $EndComp
 $Comp
-L GND #PWR013
+L GND #PWR012
 U 1 1 53D35FD0
 P 4100 6250
-F 0 "#PWR013" H 4100 6250 30  0001 C CNN
+F 0 "#PWR012" H 4100 6250 30  0001 C CNN
 F 1 "GND" H 4100 6180 30  0001 C CNN
 F 2 "" H 4100 6250 60  0000 C CNN
@@
 $EndComp
 $Comp
-L GND #PWR014
+L GND #PWR013
 U 1 1 53D36D79
 P 7300 1800
-F 0 "#PWR014" H 7300 1800 30  0001 C CNN
+F 0 "#PWR013" H 7300 1800 30  0001 C CNN
 F 1 "GND" H 7300 1730 30  0001 C CNN
 F 2 "" H 7300 1800 60  0000 C CNN
@@
 $EndComp
 $Comp
-L GND #PWR015
+L GND #PWR014
 U 1 1 53DCC533
 P 2950 6250
-F 0 "#PWR015" H 2950 6250 30  0001 C CNN
+F 0 "#PWR014" H 2950 6250 30  0001 C CNN
 F 1 "GND" H 2950 6180 30  0001 C CNN
 F 2 "" H 2950 6250 60  0000 C CNN
@@
 $EndComp
 $Comp
-L GND #PWR016
+L GND #PWR015
 U 1 1 53E0741A
 P 7000 5900
-F 0 "#PWR016" H 7000 5900 30  0001 C CNN
+F 0 "#PWR015" H 7000 5900 30  0001 C CNN
 F 1 "GND" H 7000 5830 30  0001 C CNN
 F 2 "" H 7000 5900 60  0000 C CNN
@@
 NoConn ~ 4950 5350
 $Comp
-L PWR_FLAG #FLG017
+L PWR_FLAG #FLG016
 U 1 1 53E1FC41
 P 10050 1400
-F 0 "#FLG017" H 10050 1495 30  0001 C CNN
+F 0 "#FLG016" H 10050 1495 30  0001 C CNN
 F 1 "PWR_FLAG" H 10050 1580 30  0000 C CNN
 F 2 "" H 10050 1400 60  0000 C CNN
@@
 $EndComp
 $Comp
-L GND #PWR018
+L GND #PWR017
 U 1 1 53E22E2A
 P 5350 6750
-F 0 "#PWR018" H 5350 6750 30  0001 C CNN
+F 0 "#PWR017" H 5350 6750 30  0001 C CNN
 F 1 "GND" H 5350 6680 30  0001 C CNN
 F 2 "" H 5350 6750 60  0000 C CNN
@@
 $EndComp
 $Comp
-L GND #PWR019
+L GND #PWR018
 U 1 1 53E22E4B
 P 4950 6450
-F 0 "#PWR019" H 4950 6450 30  0001 C CNN
+F 0 "#PWR018" H 4950 6450 30  0001 C CNN
 F 1 "GND" H 4950 6380 30  0001 C CNN
 F 2 "" H 4950 6450 60  0000 C CNN
@@
 NoConn ~ 5950 6350
 $Comp
-L GND #PWR020
+L GND #PWR019
 U 1 1 53E232E1
 P 4950 6250
-F 0 "#PWR020" H 4950 6250 30  0001 C CNN
+F 0 "#PWR019" H 4950 6250 30  0001 C CNN
 F 1 "GND" H 4950 6180 30  0001 C CNN
 F 2 "" H 4950 6250 60  0000 C CNN
@@
 Reset
 $Comp
-L GND #PWR021
+L GND #PWR020
 U 1 1 53E22A19
 P 7000 4950
-F 0 "#PWR021" H 7000 4950 30  0001 C CNN
+F 0 "#PWR020" H 7000 4950 30  0001 C CNN
 F 1 "GND" H 7000 4880 30  0001 C CNN
 F 2 "" H 7000 4950 60  0000 C CNN
@@
 $EndComp
 $Comp
-L GND #PWR022
+L GND #PWR021
 U 1 1 53E26458
 P 9950 1500
-F 0 "#PWR022" H 9950 1500 30  0001 C CNN
+F 0 "#PWR021" H 9950 1500 30  0001 C CNN
 F 1 "GND" H 9950 1430 30  0001 C CNN
 F 2 "" H 9950 1500 60  0000 C CNN
@@
 $EndComp
 $Comp
-L PWR_FLAG #FLG023
+L PWR_FLAG #FLG022
 U 1 1 53E267FB
 P 10050 1500
-F 0 "#FLG023" H 10050 1595 30  0001 C CNN
+F 0 "#FLG022" H 10050 1595 30  0001 C CNN
 F 1 "PWR_FLAG" H 10050 1680 30  0000 C CNN
 F 2 "" H 10050 1500 60  0000 C CNN
@@
 $EndComp
 $Comp
-L GND #PWR024
+L GND #PWR023
 U 1 1 53E234F6
 P 4150 1950
-F 0 "#PWR024" H 4150 1950 30  0001 C CNN
+F 0 "#PWR023" H 4150 1950 30  0001 C CNN
 F 1 "GND" H 4150 1880 30  0001 C CNN
 F 2 "" H 4150 1950 60  0000 C CNN
@@
 $EndComp
 $Comp
-L GND #PWR025
+L GND #PWR024
 U 1 1 53E2398F
 P 5900 1950
-F 0 "#PWR025" H 5900 1950 30  0001 C CNN
+F 0 "#PWR024" H 5900 1950 30  0001 C CNN
 F 1 "GND" H 5900 1880 30  0001 C CNN
 F 2 "" H 5900 1950 60  0000 C CNN
@@
 $EndComp
 $Comp
-L GND #PWR026
+L GND #PWR025
 U 1 1 53F32D83
 P 7900 2150
-F 0 "#PWR026" H 7900 2150 30  0001 C CNN
+F 0 "#PWR025" H 7900 2150 30  0001 C CNN
 F 1 "GND" H 7900 2080 30  0001 C CNN
 F 2 "" H 7900 2150 60  0000 C CNN
@@
 $EndComp
 $Comp
-L GND #PWR027
+L GND #PWR026
 U 1 1 53F32DAC
 P 8050 2150
-F 0 "#PWR027" H 8050 2150 30  0001 C CNN
+F 0 "#PWR026" H 8050 2150 30  0001 C CNN
 F 1 "GND" H 8050 2080 30  0001 C CNN
 F 2 "" H 8050 2150 60  0000 C CNN
@@
 $EndComp
 $Comp
-L GND #PWR028
+L GND #PWR027
 U 1 1 53F2D923
 P 7550 2550
-F 0 "#PWR028" H 7550 2550 30  0001 C CNN
+F 0 "#PWR027" H 7550 2550 30  0001 C CNN
 F 1 "GND" H 7550 2480 30  0001 C CNN
 F 2 "" H 7550 2550 60  0000 C CNN
@@
 $EndComp
 $Comp
-L GND #PWR029
+L GND #PWR028
 U 1 1 53F2D950
 P 7700 2550
-F 0 "#PWR029" H 7700 2550 30  0001 C CNN
+F 0 "#PWR028" H 7700 2550 30  0001 C CNN
 F 1 "GND" H 7700 2480 30  0001 C CNN
 F 2 "" H 7700 2550 60  0000 C CNN
@@
 $EndComp
 $Comp
-L GND #PWR030
+L GND #PWR029
 U 1 1 53F2D99F
 P 7850 2550
-F 0 "#PWR030" H 7850 2550 30  0001 C CNN
+F 0 "#PWR029" H 7850 2550 30  0001 C CNN
 F 1 "GND" H 7850 2480 30  0001 C CNN
 F 2 "" H 7850 2550 60  0000 C CNN
@@
 $EndComp
 $Comp
-L GND #PWR031
+L GND #PWR030
 U 1 1 53F2D9CC
 P 8000 2550
-F 0 "#PWR031" H 8000 2550 30  0001 C CNN
+F 0 "#PWR030" H 8000 2550 30  0001 C CNN
 F 1 "GND" H 8000 2480 30  0001 C CNN
 F 2 "" H 8000 2550 60  0000 C CNN
@@
 $EndComp
 $Comp
-L GND #PWR032
+L GND #PWR031
 U 1 1 53F2DC2E
 P 8200 2550
-F 0 "#PWR032" H 8200 2550 30  0001 C CNN
+F 0 "#PWR031" H 8200 2550 30  0001 C CNN
 F 1 "GND" H 8200 2480 30  0001 C CNN
 F 2 "" H 8200 2550 60  0000 C CNN
@@
 $EndComp
 $Comp
-L GND #PWR033
+L GND #PWR032
 U 1 1 53F2DC5D
 P 8350 2550
-F 0 "#PWR033" H 8350 2550 30  0001 C CNN
+F 0 "#PWR032" H 8350 2550 30  0001 C CNN
 F 1 "GND" H 8350 2480 30  0001 C CNN
 F 2 "" H 8350 2550 60  0000 C CNN
@@
 $EndComp
 $Comp
-L GND #PWR034
+L GND #PWR033
 U 1 1 53F2DFE3
 P 8500 2550
-F 0 "#PWR034" H 8500 2550 30  0001 C CNN
+F 0 "#PWR033" H 8500 2550 30  0001 C CNN
 F 1 "GND" H 8500 2480 30  0001 C CNN
 F 2 "" H 8500 2550 60  0000 C CNN
@@
 $EndComp
 $Comp
-L GND #PWR035
+L GND #PWR034
 U 1 1 53FEF658
 P 8950 5100
-F 0 "#PWR035" H 8950 5100 30  0001 C CNN
+F 0 "#PWR034" H 8950 5100 30  0001 C CNN
 F 1 "GND" H 8950 5030 30  0001 C CNN
 F 2 "" H 8950 5100 60  0000 C CNN
@@
 $EndComp
 $Comp
-L GND #PWR036
+L GND #PWR035
 U 1 1 5482395B
 P 7000 3250
-F 0 "#PWR036" H 7000 3250 30  0001 C CNN
+F 0 "#PWR035" H 7000 3250 30  0001 C CNN
 F 1 "GND" H 7000 3180 30  0001 C CNN
 F 2 "" H 7000 3250 60  0000 C CNN
@@
 $EndComp
 $Comp
-L GND #PWR037
+L GND #PWR036
 U 1 1 548D0F71
 P 5100 1950
-F 0 "#PWR037" H 5100 1950 30  0001 C CNN
+F 0 "#PWR036" H 5100 1950 30  0001 C CNN
 F 1 "GND" H 5100 1880 30  0001 C CNN
 F 2 "" H 5100 1950 60  0000 C CNN
@@
 $EndComp
 $Comp
-L GND #PWR038
+L GND #PWR037
 U 1 1 548D117F
 P 4450 1950
-F 0 "#PWR038" H 4450 1950 30  0001 C CNN
+F 0 "#PWR037" H 4450 1950 30  0001 C CNN
 F 1 "GND" H 4450 1880 30  0001 C CNN
 F 2 "" H 4450 1950 60  0000 C CNN
@@
 Connection ~ 6900 1400
 Connection ~ 6300 1550
+$Comp
+L TPS77033 U4
+U 1 1 54952859
+P 5900 850
+F 0 "U4" H 6050 454 60  0000 C CNN
+F 1 "TPS77033" H 5900 1050 60  0000 C CNN
+F 2 "SMD_Packages:SOT-23-5" H 5900 850 60  0001 C CNN
+F 3 "" H 5900 850 60  0000 C CNN
+	1    5900 850
+	-1   0    0    -1
+$EndComp
+$Comp
+L GND #PWR038
+U 1 1 549528C1
+P 6200 1050
+F 0 "#PWR038" H 6200 1050 30  0001 C CNN
+F 1 "GND" H 6200 980 30  0001 C CNN
+F 2 "" H 6200 1050 60  0000 C CNN
+F 3 "" H 6200 1050 60  0000 C CNN
+	1    6200 1050
+	0    -1   -1   0
+$EndComp
+NoConn ~ 5600 800
+$Comp
+L GND #PWR039
+U 1 1 549529CA
+P 5900 1300
+F 0 "#PWR039" H 5900 1300 30  0001 C CNN
+F 1 "GND" H 5900 1230 30  0001 C CNN
+F 2 "" H 5900 1300 60  0000 C CNN
+F 3 "" H 5900 1300 60  0000 C CNN
+	1    5900 1300
+	1    0    0    -1
+$EndComp
+Wire Wire Line
+	7100 1400 7100 800
+Wire Wire Line
+	7100 800  6200 800
+Connection ~ 7100 1400
+Wire Wire Line
+	5600 950  4000 950
+$Comp
+L CP C10
+U 1 1 54952BAA
+P 4250 1150
+F 0 "C10" H 4300 1250 40  0000 L CNN
+F 1 "3.3uF" H 4300 1050 40  0000 L CNN
+F 2 "SMD_Packages:SMD-1206_Pol" H 4350 1000 30  0001 C CNN
+F 3 "" H 4250 1150 300 0000 C CNN
+	1    4250 1150
+	1    0    0    -1
+$EndComp
+$Comp
+L GND #PWR040
+U 1 1 54952C3B
+P 4250 1350
+F 0 "#PWR040" H 4250 1350 30  0001 C CNN
+F 1 "GND" H 4250 1280 30  0001 C CNN
+F 2 "" H 4250 1350 60  0000 C CNN
+F 3 "" H 4250 1350 60  0000 C CNN
+	1    4250 1350
+	1    0    0    -1
+$EndComp
+Text Label 4000 950  2    60   ~ 0
+VDDX
+Text Label 7500 4450 0    60   ~ 0
+VDDX
+Connection ~ 4250 950
+$Comp
+L CONN_01X01 P19
+U 1 1 549535F9
+P 8650 2350
+F 0 "P19" H 8730 2350 40  0000 L CNN
+F 1 "CONN_1" H 8650 2405 30  0001 C CNN
+F 2 "Photodiode:THROUGHVIA" H 8650 2350 60  0001 C CNN
+F 3 "" H 8650 2350 60  0000 C CNN
+	1    8650 2350
+	0    -1   -1   0
+$EndComp
+$Comp
+L GND #PWR?
+U 1 1 5495363B
+P 8650 2550
+F 0 "#PWR?" H 8650 2550 30  0001 C CNN
+F 1 "GND" H 8650 2480 30  0001 C CNN
+F 2 "" H 8650 2550 60  0000 C CNN
+F 3 "" H 8650 2550 60  0000 C CNN
+	1    8650 2550
+	1    0    0    -1
+$EndComp
 $EndSCHEMATC

Commit message: Change PCBs to move XBee regulator and caps to the mount board. Change Vcc on mount board to take full battery voltage.
Parts:
- removed C10: 3.3uF, SMD_Packages:SMD-1206_Pol, symbol CP
- removed P19: CONN_1, Photodiode:THROUGHVIA, symbol CONN_01X01
- removed U4: TPS77033, SMD_Packages:SOT-23-5, symbol TPS77033
Connections:
- net labels removed: VDDX
- wire segments 23 -> 20
- no-connect marks 7 -> 6
Changed lines of the file:
@@
 $EndComp
 $Comp
-L GND #PWR011
+L GND #PWR012
 U 1 1 53D35BB6
 P 5350 5650
-F 0 "#PWR011" H 5350 5650 30  0001 C CNN
+F 0 "#PWR012" H 5350 5650 30  0001 C CNN
 F 1 "GND" H 5350 5580 30  0001 C CNN
 F 2 "" H 5350 5650 60  0000 C CNN
@@
 $EndComp
 $Comp
-L GND #PWR012
+L GND #PWR013
 U 1 1 53D35FD0
 P 4100 6250
-F 0 "#PWR012" H 4100 6250 30  0001 C CNN
+F 0 "#PWR013" H 4100 6250 30  0001 C CNN
 F 1 "GND" H 4100 6180 30  0001 C CNN
 F 2 "" H 4100 6250 60  0000 C CNN
@@
 $EndComp
 $Comp
-L GND #PWR013
+L GND #PWR014
 U 1 1 53D36D79
 P 7300 1800
-F 0 "#PWR013" H 7300 1800 30  0001 C CNN
+F 0 "#PWR014" H 7300 1800 30  0001 C CNN
 F 1 "GND" H 7300 1730 30  0001 C CNN
 F 2 "" H 7300 1800 60  0000 C CNN
@@
 $EndComp
 $Comp
-L GND #PWR014
+L GND #PWR015
 U 1 1 53DCC533
 P 2950 6250
-F 0 "#PWR014" H 2950 6250 30  0001 C CNN
+F 0 "#PWR015" H 2950 6250 30  0001 C CNN
 F 1 "GND" H 2950 6180 30  0001 C CNN
 F 2 "" H 2950 6250 60  0000 C CNN
@@
 $EndComp
 $Comp
-L GND #PWR015
+L GND #PWR016
 U 1 1 53E0741A
 P 7000 5900
-F 0 "#PWR015" H 7000 5900 30  0001 C CNN
+F 0 "#PWR016" H 7000 5900 30  0001 C CNN
 F 1 "GND" H 7000 5830 30  0001 C CNN
 F 2 "" H 7000 5900 60  0000 C CNN
@@
 NoConn ~ 4950 5350
 $Comp
-L PWR_FLAG #FLG016
+L PWR_FLAG #FLG017
 U 1 1 53E1FC41
 P 10050 1400
-F 0 "#FLG016" H 10050 1495 30  0001 C CNN
+F 0 "#FLG017" H 10050 1495 30  0001 C CNN
 F 1 "PWR_FLAG" H 10050 1580 30  0000 C CNN
 F 2 "" H 10050 1400 60  0000 C CNN
@@
 $EndComp
 $Comp
-L GND #PWR017
+L GND #PWR018
 U 1 1 53E22E2A
 P 5350 6750
-F 0 "#PWR017" H 5350 6750 30  0001 C CNN
+F 0 "#PWR018" H 5350 6750 30  0001 C CNN
 F 1 "GND" H 5350 6680 30  0001 C CNN
 F 2 "" H 5350 6750 60  0000 C CNN
@@
 $EndComp
 $Comp
-L GND #PWR018
+L GND #PWR019
 U 1 1 53E22E4B
 P 4950 6450
-F 0 "#PWR018" H 4950 6450 30  0001 C CNN
+F 0 "#PWR019" H 4950 6450 30  0001 C CNN
 F 1 "GND" H 4950 6380 30  0001 C CNN
 F 2 "" H 4950 6450 60  0000 C CNN
@@
 NoConn ~ 5950 6350
 $Comp
-L GND #PWR019
+L GND #PWR020
 U 1 1 53E232E1
 P 4950 6250
-F 0 "#PWR019" H 4950 6250 30  0001 C CNN
+F 0 "#PWR020" H 4950 6250 30  0001 C CNN
 F 1 "GND" H 4950 6180 30  0001 C CNN
 F 2 "" H 4950 6250 60  0000 C CNN
@@
 Reset
 $Comp
-L GND #PWR020
+L GND #PWR021
 U 1 1 53E22A19
 P 7000 4950
-F 0 "#PWR020" H 7000 4950 30  0001 C CNN
+F 0 "#PWR021" H 7000 4950 30  0001 C CNN
 F 1 "GND" H 7000 4880 30  0001 C CNN
 F 2 "" H 7000 4950 60  0000 C CNN
@@
 $EndComp
 $Comp
-L GND #PWR021
+L GND #PWR022
 U 1 1 53E26458
 P 9950 1500
-F 0 "#PWR021" H 9950 1500 30  0001 C CNN
+F 0 "#PWR022" H 9950 1500 30  0001 C CNN
 F 1 "GND" H 9950 1430 30  0001 C CNN
 F 2 "" H 9950 1500 60  0000 C CNN
@@
 $EndComp
 $Comp
-L PWR_FLAG #FLG022
+L PWR_FLAG #FLG023
 U 1 1 53E267FB
 P 10050 1500
-F 0 "#FLG022" H 10050 1595 30  0001 C CNN
+F 0 "#FLG023" H 10050 1595 30  0001 C CNN
 F 1 "PWR_FLAG" H 10050 1680 30  0000 C CNN
 F 2 "" H 10050 1500 60  0000 C CNN
@@
 $EndComp
 $Comp
-L GND #PWR023
+L GND #PWR024
 U 1 1 53E234F6
 P 4150 1950
-F 0 "#PWR023" H 4150 1950 30  0001 C CNN
+F 0 "#PWR024" H 4150 1950 30  0001 C CNN
 F 1 "GND" H 4150 1880 30  0001 C CNN
 F 2 "" H 4150 1950 60  0000 C CNN
@@
 $EndComp
 $Comp
-L GND #PWR024
+L GND #PWR025
 U 1 1 53E2398F
 P 5900 1950
-F 0 "#PWR024" H 5900 1950 30  0001 C CNN
+F 0 "#PWR025" H 5900 1950 30  0001 C CNN
 F 1 "GND" H 5900 1880 30  0001 C CNN
 F 2 "" H 5900 1950 60  0000 C CNN
@@
 $EndComp
 $Comp
-L GND #PWR025
+L GND #PWR026
 U 1 1 53F32D83
 P 7900 2150
-F 0 "#PWR025" H 7900 2150 30  0001 C CNN
+F 0 "#PWR026" H 7900 2150 30  0001 C CNN
 F 1 "GND" H 7900 2080 30  0001 C CNN
 F 2 "" H 7900 2150 60  0000 C CNN
@@
 $EndComp
 $Comp
-L GND #PWR026
+L GND #PWR027
 U 1 1 53F32DAC
 P 8050 2150
-F 0 "#PWR026" H 8050 2150 30  0001 C CNN
+F 0 "#PWR027" H 8050 2150 30  0001 C CNN
 F 1 "GND" H 8050 2080 30  0001 C CNN
 F 2 "" H 8050 2150 60  0000 C CNN
@@
 $EndComp
 $Comp
-L GND #PWR027
+L GND #PWR028
 U 1 1 53F2D923
 P 7550 2550
-F 0 "#PWR027" H 7550 2550 30  0001 C CNN
+F 0 "#PWR028" H 7550 2550 30  0001 C CNN
 F 1 "GND" H 7550 2480 30  0001 C CNN
 F 2 "" H 7550 2550 60  0000 C CNN
@@
 $EndComp
 $Comp
-L GND #PWR028
+L GND #PWR029
 U 1 1 53F2D950
 P 7700 2550
-F 0 "#PWR028" H 7700 2550 30  0001 C CNN
+F 0 "#PWR029" H 7700 2550 30  0001 C CNN
 F 1 "GND" H 7700 2480 30  0001 C CNN
 F 2 "" H 7700 2550 60  0000 C CNN
@@
 $EndComp
 $Comp
-L GND #PWR029
+L GND #PWR030
 U 1 1 53F2D99F
 P 7850 2550
-F 0 "#PWR029" H 7850 2550 30  0001 C CNN
+F 0 "#PWR030" H 7850 2550 30  0001 C CNN
 F 1 "GND" H 7850 2480 30  0001 C CNN
 F 2 "" H 7850 2550 60  0000 C CNN
@@
 $EndComp
 $Comp
-L GND #PWR030
+L GND #PWR031
 U 1 1 53F2D9CC
 P 8000 2550
-F 0 "#PWR030" H 8000 2550 30  0001 C CNN
+F 0 "#PWR031" H 8000 2550 30  0001 C CNN
 F 1 "GND" H 8000 2480 30  0001 C CNN
 F 2 "" H 8000 2550 60  0000 C CNN
@@
 $EndComp
 $Comp
-L GND #PWR031
+L GND #PWR032
 U 1 1 53F2DC2E
 P 8200 2550
-F 0 "#PWR031" H 8200 2550 30  0001 C CNN
+F 0 "#PWR032" H 8200 2550 30  0001 C CNN
 F 1 "GND" H 8200 2480 30  0001 C CNN
 F 2 "" H 8200 2550 60  0000 C CNN
@@
 $EndComp
 $Comp
-L GND #PWR032
+L GND #PWR033
 U 1 1 53F2DC5D
 P 8350 2550
-F 0 "#PWR032" H 8350 2550 30  0001 C CNN
+F 0 "#PWR033" H 8350 2550 30  0001 C CNN
 F 1 "GND" H 8350 2480 30  0001 C CNN
 F 2 "" H 8350 2550 60  0000 C CNN
@@
 $EndComp
 $Comp
-L GND #PWR033
+L GND #PWR034
 U 1 1 53F2DFE3
 P 8500 2550
-F 0 "#PWR033" H 8500 2550 30  0001 C CNN
+F 0 "#PWR034" H 8500 2550 30  0001 C CNN
 F 1 "GND" H 8500 2480 30  0001 C CNN
 F 2 "" H 8500 2550 60  0000 C CNN
@@
 $EndComp
 $Comp
-L GND #PWR034
+L GND #PWR035
 U 1 1 53FEF658
 P 8950 5100
-F 0 "#PWR034" H 8950 5100 30  0001 C CNN
+F 0 "#PWR035" H 8950 5100 30  0001 C CNN
 F 1 "GND" H 8950 5030 30  0001 C CNN
 F 2 "" H 8950 5100 60  0000 C CNN
@@
 $EndComp
 $Comp
-L GND #PWR035
+L GND #PWR036
 U 1 1 5482395B
 P 7000 3250
-F 0 "#PWR035" H 7000 3250 30  0001 C CNN
+F 0 "#PWR036" H 7000 3250 30  0001 C CNN
 F 1 "GND" H 7000 3180 30  0001 C CNN
 F 2 "" H 7000 3250 60  0000 C CNN
@@
 $EndComp
 $Comp
-L GND #PWR036
+L GND #PWR037
 U 1 1 548D0F71
 P 5100 1950
-F 0 "#PWR036" H 5100 1950 30  0001 C CNN
+F 0 "#PWR037" H 5100 1950 30  0001 C CNN
 F 1 "GND" H 5100 1880 30  0001 C CNN
 F 2 "" H 5100 1950 60  0000 C CNN
@@
 $EndComp
 $Comp
-L GND #PWR037
+L GND #PWR038
 U 1 1 548D117F
 P 4450 1950
-F 0 "#PWR037" H 4450 1950 30  0001 C CNN
+F 0 "#PWR038" H 4450 1950 30  0001 C CNN
 F 1 "GND" H 4450 1880 30  0001 C CNN
 F 2 "" H 4450 1950 60  0000 C CNN
@@
 Connection ~ 6900 1400
 Connection ~ 6300 1550
-$Comp
-L TPS77033 U4
-U 1 1 54952859
-P 5900 850
-F 0 "U4" H 6050 454 60  0000 C CNN
-F 1 "TPS77033" H 5900 1050 60  0000 C CNN
-F 2 "SMD_Packages:SOT-23-5" H 5900 850 60  0001 C CNN
-F 3 "" H 5900 850 60  0000 C CNN
-	1    5900 850
-	-1   0    0    -1
-$EndComp
-$Comp
-L GND #PWR038
-U 1 1 549528C1
-P 6200 1050
-F 0 "#PWR038" H 6200 1050 30  0001 C CNN
-F 1 "GND" H 6200 980 30  0001 C CNN
-F 2 "" H 6200 1050 60  0000 C CNN
-F 3 "" H 6200 1050 60  0000 C CNN
-	1    6200 1050
-	0    -1   -1   0
-$EndComp
-NoConn ~ 5600 800
-$Comp
-L GND #PWR039
-U 1 1 549529CA
-P 5900 1300
-F 0 "#PWR039" H 5900 1300 30  0001 C CNN
-F 1 "GND" H 5900 1230 30  0001 C CNN
-F 2 "" H 5900 1300 60  0000 C CNN
-F 3 "" H 5900 1300 60  0000 C CNN
-	1    5900 1300
-	1    0    0    -1
-$EndComp
-Wire Wire Line
-	7100 1400 7100 800
-Wire Wire Line
-	7100 800  6200 800
-Connection ~ 7100 1400
-Wire Wire Line
-	5600 950  4000 950
-$Comp
-L CP C10
-U 1 1 54952BAA
-P 4250 1150
-F 0 "C10" H 4300 1250 40  0000 L CNN
-F 1 "3.3uF" H 4300 1050 40  0000 L CNN
-F 2 "SMD_Packages:SMD-1206_Pol" H 4350 1000 30  0001 C CNN
-F 3 "" H 4250 1150 300 0000 C CNN
-	1    4250 1150
-	1    0    0    -1
-$EndComp
-$Comp
-L GND #PWR040
-U 1 1 54952C3B
-P 4250 1350
-F 0 "#PWR040" H 4250 1350 30  0001 C CNN
-F 1 "GND" H 4250 1280 30  0001 C CNN
-F 2 "" H 4250 1350 60  0000 C CNN
-F 3 "" H 4250 1350 60  0000 C CNN
-	1    4250 1350
-	1    0    0    -1
-$EndComp
-Text Label 4000 950  2    60   ~ 0
-VDDX
 Text Label 7500 4450 0    60   ~ 0
-VDDX
-Connection ~ 4250 950
-$Comp
-L CONN_01X01 P19
-U 1 1 549535F9
-P 8650 2350
-F 0 "P19" H 8730 2350 40  0000 L CNN
-F 1 "CONN_1" H 8650 2405 30  0001 C CNN
-F 2 "Photodiode:THROUGHVIA" H 8650 2350 60  0001 C CNN
-F 3 "" H 8650 2350 60  0000 C CNN
-	1    8650 2350
-	0    -1   -1   0
-$EndComp
-$Comp
-L GND #PWR?
-U 1 1 5495363B
-P 8650 2550
-F 0 "#PWR?" H 8650 2550 30  0001 C CNN
-F 1 "GND" H 8650 2480 30  0001 C CNN
-F 2 "" H 8650 2550 60  0000 C CNN
-F 3 "" H 8650 2550 60  0000 C CNN
-	1    8650 2550
-	1    0    0    -1
-$EndComp
+Battery
 $EndSCHEMATC
