File: Kicad-TestBoard/Kicad-TestBoard.sch (KiCad schematic (older format))
At the start: 35 parts, among them CON1 Power 6V-12V, J2 DB9 RS-232 Female, P1 Power 6V-12V, P2 Debug, P3 Debug, P4 Arduino Digital Input, P5 AVR Programmer, P6 RS-232, Q1 Association, Q2 On_Sleep, Q3 Commissioning, SW1 Reset, SW2 Commissioning, U1 78L05, U1 MAX232

Commit message: Addition of PCB layout to testboard with footprints taken mainly from Kicad GitHub repository. Not yet routed
Parts:
- C1: footprint (none) -> Testboard:C_Disc_D3_P2.5
- C2: footprint (none) -> Testboard:C_Radial_D5_L11_P2.5
- C3: renamed from C4; footprint (none) -> Testboard:C_Radial_D5_L11_P2.5
- C4: renamed from C5; footprint (none) -> Testboard:C_Radial_D5_L11_P2.5
- C5: renamed from C6; footprint (none) -> Testboard:C_Radial_D5_L11_P2.5
- C6: renamed from C7; footprint (none) -> Testboard:C_Radial_D5_L11_P2.5
- CON1: footprint (none) -> Testboard:BARREL_JACK
- D1, D2, D3: footprint (none) -> Testboard:LED-5MM
- J1: renamed from J2; footprint (none) -> Testboard:DB9FD
- P1: footprint (none) -> Testboard:PINHEAD1-2
- P2: footprint (none) -> Testboard:pin_header_2mm_2x6
- P3: footprint (none) -> Testboard:IDC_Header_Straight_12pins
- P4: footprint (none) -> Testboard:PINHEAD1-3
- P5: footprint (none) -> Testboard:PINHEAD1-6
- P6: footprint (none) -> Testboard:PINHEAD1-4
- Q1, Q2, Q3: footprint (none) -> Testboard:TO-92_Molded_Narrow
- R1, R2, R3, R4, R5, R6, R7, R8: footprint (none) -> Testboard:Resistor_Horizontal_RM10mm
- SW1, SW2: footprint (none) -> Testboard:SW_PUSH_SMALL
- U1: footprint (none) -> Testboard:TO-220
- U2: renamed from U1; footprint (none) -> Testboard:DIP-16_W7.62mm; symbol MAX232 -> MAX232-RESCUE-Kicad-TestBoard
- W1, W2: footprint (none) -> Testboard:SIL-1
- W3: renamed from W1; footprint (none) -> Testboard:SIL-2
Connections:
- wire segments 83 -> 64
Other:
- moved on the sheet: C2, U1

Commit message: Completion of test board. The 0.1" 12-pin debug connector removed as unnecessary and too complicating for the layout. PB switches adapted to smaller more common version available locally.
Parts:
- removed P3: Debug, Testboard:IDC_Header_Straight_12pins, symbol CONN_02X06
- P2: footprint Testboard:pin_header_2mm_2x6 -> Testboard:pin_header_2mm_2x6_shrouded
- P4: value Arduino Digital Input -> Arduino
- U1: symbol 7805 -> 7805-RESCUE-Kicad-TestBoard
Connections:
- net labels removed: Association
- wire segments 64 -> 59
- no-connect marks 0 -> 7
Other:
- moved on the sheet: D1, D2, D3, P1, Q1, Q2, Q3, R1, R2, R3, R4, R5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

Commit message: Testboard. Correct some footprint errors and change drill sizes to regular metric.
Parts:
- SW1, SW2: footprint Testboard:SW_PUSH_SMALL -> Testboard:SW_PUSH_TINY
- U1: footprint Testboard:TO-220 -> Testboard:TO-92_Molded_Narrow
Connections:
- wire segments 59 -> 48
Changed lines of the file:
@@
 F 0 "U1" H 3400 2715 50  0000 C CNN
 F 1 "78L05" H 3400 2624 50  0000 C CNN
-F 2 "Testboard:TO-220" H 3400 2400 50  0001 C CNN
+F 2 "Testboard:TO-92_Molded_Narrow" H 3400 2400 50  0001 C CNN
 F 3 "" H 3400 2400 50  0000 C CNN
 	1    3400 2400
@@
 F 0 "SW1" H 1300 3655 50  0000 C CNN
 F 1 "Reset" H 1300 3564 50  0000 C CNN
-F 2 "Testboard:SW_PUSH_SMALL" H 1300 3400 50  0001 C CNN
+F 2 "Testboard:SW_PUSH_TINY" H 1300 3400 50  0001 C CNN
 F 3 "" H 1300 3400 50  0000 C CNN
 	1    1300 3400
@@
 $EndComp
 $Comp
-L Earth #PWR04
+L Earth #PWR03
 U 1 1 5757B92E
 P 1000 3400
-F 0 "#PWR04" H 1000 3150 50  0001 C CNN
+F 0 "#PWR03" H 1000 3150 50  0001 C CNN
 F 1 "Earth" H 1000 3250 50  0001 C CNN
 F 2 "" H 1000 3400 50  0000 C CNN
@@
 F 0 "SW2" H 1300 4205 50  0000 C CNN
 F 1 "Commissioning" H 1300 4114 50  0000 C CNN
-F 2 "Testboard:SW_PUSH_SMALL" H 1300 3950 50  0001 C CNN
+F 2 "Testboard:SW_PUSH_TINY" H 1300 3950 50  0001 C CNN
 F 3 "" H 1300 3950 50  0000 C CNN
 	1    1300 3950
@@
 $EndComp
 $Comp
-L Earth #PWR05
+L Earth #PWR04
 U 1 1 5757BB82
 P 1000 3950
-F 0 "#PWR05" H 1000 3700 50  0001 C CNN
+F 0 "#PWR04" H 1000 3700 50  0001 C CNN
 F 1 "Earth" H 1000 3800 50  0001 C CNN
 F 2 "" H 1000 3950 50  0000 C CNN
@@
 $EndComp
 $Comp
-L Earth #PWR06
+L Earth #PWR05
 U 1 1 5757BFBE
 P 4600 2450
-F 0 "#PWR06" H 4600 2200 50  0001 C CNN
+F 0 "#PWR05" H 4600 2200 50  0001 C CNN
 F 1 "Earth" H 4600 2300 50  0001 C CNN
 F 2 "" H 4600 2450 50  0000 C CNN
@@
 $EndComp
 $Comp
-L Earth #PWR07
+L Earth #PWR06
 U 1 1 5757C491
 P 4150 3400
-F 0 "#PWR07" H 4150 3150 50  0001 C CNN
+F 0 "#PWR06" H 4150 3150 50  0001 C CNN
 F 1 "Earth" H 4150 3250 50  0001 C CNN
 F 2 "" H 4150 3400 50  0000 C CNN
@@
 $EndComp
 $Comp
-L Earth #PWR08
+L Earth #PWR07
 U 1 1 5757CADB
 P 4150 3750
-F 0 "#PWR08" H 4150 3500 50  0001 C CNN
+F 0 "#PWR07" H 4150 3500 50  0001 C CNN
 F 1 "Earth" H 4150 3600 50  0001 C CNN
 F 2 "" H 4150 3750 50  0000 C CNN
@@
 $EndComp
 $Comp
-L Earth #PWR09
+L Earth #PWR08
 U 1 1 5757E113
 P 8950 3300
-F 0 "#PWR09" H 8950 3050 50  0001 C CNN
+F 0 "#PWR08" H 8950 3050 50  0001 C CNN
 F 1 "Earth" H 8950 3150 50  0001 C CNN
 F 2 "" H 8950 3300 50  0000 C CNN
@@
 $EndComp
 $Comp
-L VCC #PWR010
+L VCC #PWR09
 U 1 1 5757E882
 P 3800 2350
-F 0 "#PWR010" H 3800 2200 50  0001 C CNN
+F 0 "#PWR09" H 3800 2200 50  0001 C CNN
 F 1 "VCC" H 3817 2523 50  0000 C CNN
 F 2 "" H 3800 2350 50  0000 C CNN
@@
 $EndComp
 $Comp
-L VCC #PWR011
+L VCC #PWR010
 U 1 1 5757E8CC
 P 6350 3150
-F 0 "#PWR011" H 6350 3000 50  0001 C CNN
+F 0 "#PWR010" H 6350 3000 50  0001 C CNN
 F 1 "VCC" H 6367 3323 50  0000 C CNN
 F 2 "" H 6350 3150 50  0000 C CNN
@@
 $EndComp
 $Comp
-L Earth #PWR012
+L Earth #PWR011
 U 1 1 5757EBCE
 P 3850 6200
-F 0 "#PWR012" H 3850 5950 50  0001 C CNN
+F 0 "#PWR011" H 3850 5950 50  0001 C CNN
 F 1 "Earth" H 3850 6050 50  0001 C CNN
 F 2 "" H 3850 6200 50  0000 C CNN
@@
 $EndComp
 $Comp
-L VCC #PWR013
+L VCC #PWR012
 U 1 1 5757EC33
 P 3850 5100
-F 0 "#PWR013" H 3850 4950 50  0001 C CNN
+F 0 "#PWR012" H 3850 4950 50  0001 C CNN
 F 1 "VCC" H 3867 5273 50  0000 C CNN
 F 2 "" H 3850 5100 50  0000 C CNN
@@
 $EndComp
 $Comp
-L VCC #PWR014
+L VCC #PWR013
 U 1 1 5758127D
 P 2800 5100
-F 0 "#PWR014" H 2800 4950 50  0001 C CNN
+F 0 "#PWR013" H 2800 4950 50  0001 C CNN
 F 1 "VCC" H 2817 5273 50  0000 C CNN
 F 2 "" H 2800 5100 50  0000 C CNN
@@
 $EndComp
 $Comp
-L Earth #PWR015
+L Earth #PWR014
 U 1 1 5758197B
 P 2800 6200
-F 0 "#PWR015" H 2800 5950 50  0001 C CNN
+F 0 "#PWR014" H 2800 5950 50  0001 C CNN
 F 1 "Earth" H 2800 6050 50  0001 C CNN
 F 2 "" H 2800 6200 50  0000 C CNN
@@
 $EndComp
 $Comp
-L VCC #PWR016
+L VCC #PWR015
 U 1 1 57582756
 P 1750 5100
-F 0 "#PWR016" H 1750 4950 50  0001 C CNN
+F 0 "#PWR015" H 1750 4950 50  0001 C CNN
 F 1 "VCC" H 1767 5273 50  0000 C CNN
 F 2 "" H 1750 5100 50  0000 C CNN
@@
 $EndComp
 $Comp
-L Earth #PWR017
+L Earth #PWR016
 U 1 1 57582A1D
 P 1750 6200
-F 0 "#PWR017" H 1750 5950 50  0001 C CNN
+F 0 "#PWR016" H 1750 5950 50  0001 C CNN
 F 1 "Earth" H 1750 6050 50  0001 C CNN
 F 2 "" H 1750 6200 50  0000 C CNN
@@
 $EndComp
 Wire Wire Line
-	2050 2350 2250 2350
-Wire Wire Line
-	2250 2350 2400 2350
-Wire Wire Line
-	2400 2350 2550 2350
-Wire Wire Line
-	2550 2350 2850 2350
-Wire Wire Line
-	2850 2350 3000 2350
+	2050 2350 3000 2350
 Wire Wire Line
 	2000 1850 2400 1850
@@
 	2050 3700 2050 5700
 Wire Wire Line
-	2850 3300 3350 3300
-Wire Wire Line
-	3350 3300 4150 3300
+	2850 3300 4150 3300
 Wire Wire Line
 	2850 3400 4000 3400
@@
 Connection ~ 2200 3400
 Wire Wire Line
-	1600 3400 2200 3400
-Wire Wire Line
-	2200 3400 2350 3400
-Wire Wire Line
-	1600 3950 3300 3950
-Wire Wire Line
-	3300 3950 3550 3950
+	1600 3400 2350 3400
+Wire Wire Line
+	1600 3950 3550 3950
 Connection ~ 3350 3300
 Wire Wire Line
@@
 $EndComp
 $Comp
-L Earth #PWR018
+L Earth #PWR017
 U 1 1 57583CC1
 P 7450 3950
-F 0 "#PWR018" H 7450 3700 50  0001 C CNN
+F 0 "#PWR017" H 7450 3700 50  0001 C CNN
 F 1 "Earth" H 7450 3800 50  0001 C CNN
 F 2 "" H 7450 3950 50  0000 C CNN
@@
 $EndComp
 Wire Wire Line
-	3200 4850 4700 4850
-Wire Wire Line
-	4700 4850 4850 4850
-$Comp
-L Earth #PWR019
+	3200 4850 4850 4850
+$Comp
+L Earth #PWR018
 U 1 1 5758448E
 P 4700 5150
-F 0 "#PWR019" H 4700 4900 50  0001 C CNN
+F 0 "#PWR018" H 4700 4900 50  0001 C CNN
 F 1 "Earth" H 4700 5000 50  0001 C CNN
 F 2 "" H 4700 5150 50  0000 C CNN
@@
 $EndComp
 $Comp
-L Earth #PWR020
+L Earth #PWR019
 U 1 1 57584E0E
 P 2550 2650
-F 0 "#PWR020" H 2550 2400 50  0001 C CNN
+F 0 "#PWR019" H 2550 2400 50  0001 C CNN
 F 1 "Earth" H 2550 2500 50  0001 C CNN
 F 2 "" H 2550 2650 50  0000 C CNN
@@
 $EndComp
 $Comp
-L Earth #PWR021
+L Earth #PWR020
 U 1 1 57584E82
 P 2850 2650
-F 0 "#PWR021" H 2850 2400 50  0001 C CNN
+F 0 "#PWR020" H 2850 2400 50  0001 C CNN
 F 1 "Earth" H 2850 2500 50  0001 C CNN
 F 2 "" H 2850 2650 50  0000 C CNN
@@
 Connection ~ 2550 2350
 $Comp
-L VCC #PWR022
+L VCC #PWR021
 U 1 1 575852C0
 P 4150 4250
-F 0 "#PWR022" H 4150 4100 50  0001 C CNN
+F 0 "#PWR021" H 4150 4100 50  0001 C CNN
 F 1 "VCC" V 4168 4377 50  0000 L CNN
 F 2 "" H 4150 4250 50  0000 C CNN
@@
 $EndComp
 $Comp
-L Earth #PWR023
+L Earth #PWR022
 U 1 1 5758599D
 P 7450 4250
-F 0 "#PWR023" H 7450 4000 50  0001 C CNN
+F 0 "#PWR022" H 7450 4000 50  0001 C CNN
 F 1 "Earth" H 7450 4100 50  0001 C CNN
 F 2 "" H 7450 4250 50  0000 C CNN
@@
 $EndComp
 Wire Wire Line
-	8150 3500 8150 4450
-Wire Wire Line
-	8150 4450 8150 4850
+	8150 3500 8150 4850
 Wire Wire Line
 	8150 4850 7150 4850
@@
 	8000 4650 7150 4650
 Wire Wire Line
-	8000 3400 8000 4250
-Wire Wire Line
-	8000 4250 8000 4650
+	8000 3400 8000 4650
 Wire Wire Line
 	8000 3400 8950 3400
@@
 Connection ~ 8150 4450
 $Comp
-L Earth #PWR025
+L Earth #PWR023
 U 1 1 5758BB8A
 P 8750 4850
-F 0 "#PWR025" H 8750 4600 50  0001 C CNN
+F 0 "#PWR023" H 8750 4600 50  0001 C CNN
 F 1 "Earth" H 8750 4700 50  0001 C CNN
 F 2 "" H 8750 4850 50  0000 C CNN
@@
 	8750 4050 8600 4050
 Wire Wire Line
-	8600 4050 8600 4150
-Wire Wire Line
-	8600 4150 8600 4650
+	8600 4050 8600 4650
 Wire Wire Line
 	8600 4150 8750 4150
@@
 Connection ~ 2250 2350
 $Comp
-L Earth #PWR026
+L Earth #PWR024
 U 1 1 57579A7B
 P 2050 2550
-F 0 "#PWR026" H 2050 2300 50  0001 C CNN
+F 0 "#PWR024" H 2050 2300 50  0001 C CNN
 F 1 "Earth" H 2050 2400 50  0001 C CNN
 F 2 "" H 2050 2550 50  0000 C CNN
@@
 F 3 "" H 1750 2450 50  0000 C CNN
 	1    1750 2450
-	1    0    0    1
+	1    0    0    -1
 $EndComp
 $Comp
@@
 NoConn ~ 5550 5050
 NoConn ~ 5550 4650
-Wire Wire Line
-	2050 2450 2050 2350
-Connection ~ 2050 2350
+Connection ~ 2050 2550
 Connection ~ 4700 4850
 NoConn ~ 4150 3200
 $Comp
-L Earth #PWR?
+L Earth #PWR025
 U 1 1 57635380
 P 2350 3800
-F 0 "#PWR?" H 2350 3550 50  0001 C CNN
+F 0 "#PWR025" H 2350 3550 50  0001 C CNN
 F 1 "Earth" H 2350 3650 50  0001 C CNN
 F 2 "" H 2350 3800 50  0000 C CNN
@@
 	2050 3700 2350 3700
 $Comp
-L Earth #PWR?
+L Earth #PWR026
 U 1 1 57637FFA
 P 6350 5550
-F 0 "#PWR?" H 6350 5300 50  0001 C CNN
+F 0 "#PWR026" H 6350 5300 50  0001 C CNN
 F 1 "Earth" H 6350 5400 50  0001 C CNN
 F 2 "" H 6350 5550 50  0000 C CNN
@@
 	1    0    0    -1
 $EndComp
+Wire Wire Line
+	2050 2450 2050 2550
 $EndSCHEMATC

Commit message: Update of Testboard PCB and generation of gerbers.
Parts:
- Q1, Q2, Q3, U1: footprint Testboard:TO-92_Molded_Narrow -> Testboard:TO-92_Molded_Wide
Changed lines of the file:
@@
 F 0 "U1" H 3400 2715 50  0000 C CNN
 F 1 "78L05" H 3400 2624 50  0000 C CNN
-F 2 "Testboard:TO-92_Molded_Narrow" H 3400 2400 50  0001 C CNN
+F 2 "Testboard:TO-92_Molded_Wide" H 3400 2400 50  0001 C CNN
 F 3 "" H 3400 2400 50  0000 C CNN
 	1    3400 2400
@@
 F 0 "Q3" H 3941 6046 50  0000 L CNN
 F 1 "Commissioning" H 3941 5955 50  0000 L CNN
-F 2 "Testboard:TO-92_Molded_Narrow" H 3950 6100 50  0001 C CNN
+F 2 "Testboard:TO-92_Molded_Wide" H 3950 6100 50  0001 C CNN
 F 3 "" H 3750 6000 50  0000 C CNN
 	1    3750 6000
@@
 F 0 "Q2" H 3091 6046 50  0000 L CNN
 F 1 "On_Sleep" H 3091 5955 50  0000 L CNN
-F 2 "Testboard:TO-92_Molded_Narrow" H 3100 6100 50  0001 C CNN
+F 2 "Testboard:TO-92_Molded_Wide" H 3100 6100 50  0001 C CNN
 F 3 "" H 2900 6000 50  0000 C CNN
 	1    2900 6000
@@
 F 0 "Q1" H 2041 6046 50  0000 L CNN
 F 1 "Association" H 2041 5955 50  0000 L CNN
-F 2 "Testboard:TO-92_Molded_Narrow" H 2050 6100 50  0001 C CNN
+F 2 "Testboard:TO-92_Molded_Wide" H 2050 6100 50  0001 C CNN
 F 3 "" H 1850 6000 50  0000 C CNN
 	1    1850 6000

Commit message: Testboard: repair schematic by removing repair library and replacing symbols with those present in Kicad.
Parts:
- U1: symbol 7805-RESCUE-Kicad-TestBoard -> 7805
- U2: symbol MAX232-RESCUE-Kicad-TestBoard -> MAX232
Connections:
- wire segments 48 -> 66
Other:
- moved on the sheet: C3, C4, C5, C6, D1, D2, D3, Q1, Q2, Q3, R1, R2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
